File: logic-probe/logic-probe.sch (KiCad schematic (older format))
At the start: 16 parts

Commit message: first drawn schematic
Parts:
- added D?: LED, symbol Device:LED
- added J?: Conn_01x01_Male, symbol Connector:Conn_01x01_Male
- added R? (x4): R, symbol Device:R
Connections:
- net GND: now also Q?.3 (C2), R?.2
- net VDD: now reaches R?.1
- net VDD: now also Q?.6 (C1), R?.1
- net Vp: now reaches R?.1, R?.2
- net at U?.3 (+): now also Q?.4 (E2), R?.2
- net Vn: now reaches U?.5 (+)
- net Vn: now also R?.1, R?.2
- net at U?.6 (_): now also Q?.1 (E1), R?.1
- net at R?.1: now also D?.1 (K); no longer U?.4
- net at Q?.2 (B1): now also R?.1
- net at Q?.5 (B2): now also R?.1
- new net: D?.2 (A), U?.4
- new net: J?.1 (Pin_1), R?.2, R?.2
Other:
- moved on the sheet: Q?A, Q?B, R?
